File: Kicad/dev-board/dev-board.sch (KiCad schematic (older format))
At the start: 60 parts, among them J1 Conn_01x01_Male, J10 Conn_01x03_Male, J11 Conn_01x03_Male, J12 Conn_01x01_Male, J13 Conn_01x04_Male, J14 Conn_01x01_Male, J15 Conn_01x03_Male, J16 Conn_01x06_Male, J2 Conn_01x04_Male, J3 Conn_01x02_Male, J4 Conn_01x02_Male, J5 Conn_01x02_Male, J6 Conn_01x02_Male, J7 Conn_01x04_Male, J8 Conn_01x03_Male, J9 Conn_01x03_Male, Q1 2N2219, SW1 SW_DIP_x04, SW2 SW_SPDT, SW3 SW_SPDT, SW4 SW_Push, SW5 SW_Push, SW6 SW_Push, SW7 SW_Push, SW8 Rotary_Encoder_Switch, U1 NE555P

Commit message: PCB final step
Parts:
- removed J1, J12, J14: Conn_01x01_Male, Connector_PinHeader_2.54mm:PinHeader_1x01_P2.54mm_Vertical, symbol Connector:Conn_01x01_Male
- added C2: C, Capacitor_SMD:C_0805_2012Metric_Pad1.15x1.40mm_HandSolder, symbol Device:C
- added J1: Conn_01x03_Male, Connector_PinHeader_2.54mm:PinHeader_1x03_P2.54mm_Vertical, symbol Connector:Conn_01x03_Male
- J2: footprint Connector_PinHeader_2.54mm:PinHeader_1x04_P2.54mm_Vertical -> Connector_JST:JST_XH_B4B-XH-A_1x04_P2.50mm_Vertical
- R1, R10, R11, R12, R13, R14, R15, R16, R17, R18, R19, R2, R20, R21, R3, R4, R6, R7, R8, R9: footprint Resistor_SMD:R_0815_2038Metric_Pad1.53x4.00mm_HandSolder -> Resistor_SMD:R_0805_2012Metric_Pad1.15x1.40mm_HandSolder
- RV1, RV2: footprint (none) -> Potentiometer_THT:Potentiometer_Bourns_3386P_Vertical
Connections:
- net GND: now also C2.2
- net light_sensor_pin: now reaches R5.2, R6.2
- net light_sensor_pin: now also J1.1 (Pin_1)
- net timer_pin: now reaches R11.2, U1.3 (Q)
- net timer_pin: now also J1.3 (Pin_3)
- net at U1.5 (CV): now also C2.1
- net at R1.2: now also J1.2 (Pin_2)
- no-connect marks 2 -> 1
Changed lines of the file:
@@
 F 0 "RV1" H 1181 6896 50  0000 R CNN
 F 1 "R_POT" H 1181 6805 50  0000 R CNN
-F 2 "" H 1250 6850 50  0001 C CNN
+F 2 "Potentiometer_THT:Potentiometer_Bourns_3386P_Vertical" H 1250 6850 50  0001 C CNN
 F 3 "~" H 1250 6850 50  0001 C CNN
 	1    1250 6850
@@
 F 0 "RV2" H 1931 6896 50  0000 R CNN
 F 1 "R_POT" H 1931 6805 50  0000 R CNN
-F 2 "" H 2000 6850 50  0001 C CNN
+F 2 "Potentiometer_THT:Potentiometer_Bourns_3386P_Vertical" H 2000 6850 50  0001 C CNN
 F 3 "~" H 2000 6850 50  0001 C CNN
 	1    2000 6850
@@
 F 0 "R17" V 9650 2600 50  0000 L CNN
 F 1 "R" V 9650 2500 50  0000 L CNN
-F 2 "Resistor_SMD:R_0815_2038Metric_Pad1.53x4.00mm_HandSolder" V 9480 2600 50  0001 C CNN
+F 2 "Resistor_SMD:R_0805_2012Metric_Pad1.15x1.40mm_HandSolder" V 9480 2600 50  0001 C CNN
 F 3 "~" H 9550 2600 50  0001 C CNN
 	1    9550 2600
@@
 F 0 "R18" V 9650 2900 50  0000 L CNN
 F 1 "R" V 9650 2800 50  0000 L CNN
-F 2 "Resistor_SMD:R_0815_2038Metric_Pad1.53x4.00mm_HandSolder" V 9480 2900 50  0001 C CNN
+F 2 "Resistor_SMD:R_0805_2012Metric_Pad1.15x1.40mm_HandSolder" V 9480 2900 50  0001 C CNN
 F 3 "~" H 9550 2900 50  0001 C CNN
 	1    9550 2900
@@
 F 0 "R19" V 9650 3200 50  0000 L CNN
 F 1 "R" V 9650 3100 50  0000 L CNN
-F 2 "Resistor_SMD:R_0815_2038Metric_Pad1.53x4.00mm_HandSolder" V 9480 3200 50  0001 C CNN
+F 2 "Resistor_SMD:R_0805_2012Metric_Pad1.15x1.40mm_HandSolder" V 9480 3200 50  0001 C CNN
 F 3 "~" H 9550 3200 50  0001 C CNN
 	1    9550 3200
@@
 F 0 "R15" V 9650 2000 50  0000 L CNN
 F 1 "R" V 9650 1900 50  0000 L CNN
-F 2 "Resistor_SMD:R_0815_2038Metric_Pad1.53x4.00mm_HandSolder" V 9480 2000 50  0001 C CNN
+F 2 "Resistor_SMD:R_0805_2012Metric_Pad1.15x1.40mm_HandSolder" V 9480 2000 50  0001 C CNN
 F 3 "~" H 9550 2000 50  0001 C CNN
 	1    9550 2000
@@
 F 0 "R16" V 9650 2300 50  0000 L CNN
 F 1 "R" V 9650 2200 50  0000 L CNN
-F 2 "Resistor_SMD:R_0815_2038Metric_Pad1.53x4.00mm_HandSolder" V 9480 2300 50  0001 C CNN
+F 2 "Resistor_SMD:R_0805_2012Metric_Pad1.15x1.40mm_HandSolder" V 9480 2300 50  0001 C CNN
 F 3 "~" H 9550 2300 50  0001 C CNN
 	1    9550 2300
@@
 F 0 "R2" H 2020 1446 50  0000 L CNN
 F 1 "R" H 2020 1355 50  0000 L CNN
-F 2 "Resistor_SMD:R_0815_2038Metric_Pad1.53x4.00mm_HandSolder" V 1880 1400 50  0001 C CNN
+F 2 "Resistor_SMD:R_0805_2012Metric_Pad1.15x1.40mm_HandSolder" V 1880 1400 50  0001 C CNN
 F 3 "~" H 1950 1400 50  0001 C CNN
 	1    1950 1400
@@
 F 0 "R20" V 9650 4900 50  0000 L CNN
 F 1 "R" V 9650 4800 50  0000 L CNN
-F 2 "Resistor_SMD:R_0815_2038Metric_Pad1.53x4.00mm_HandSolder" V 9480 4900 50  0001 C CNN
+F 2 "Resistor_SMD:R_0805_2012Metric_Pad1.15x1.40mm_HandSolder" V 9480 4900 50  0001 C CNN
 F 3 "~" H 9550 4900 50  0001 C CNN
 	1    9550 4900
@@
 F 0 "R13" V 9450 4900 50  0000 L CNN
 F 1 "R" V 9450 4800 50  0000 L CNN
-F 2 "Resistor_SMD:R_0815_2038Metric_Pad1.53x4.00mm_HandSolder" V 9280 4900 50  0001 C CNN
+F 2 "Resistor_SMD:R_0805_2012Metric_Pad1.15x1.40mm_HandSolder" V 9280 4900 50  0001 C CNN
 F 3 "~" H 9350 4900 50  0001 C CNN
 	1    9350 4900
@@
 F 0 "R21" V 9850 4900 50  0000 L CNN
 F 1 "R" V 9850 4800 50  0000 L CNN
-F 2 "Resistor_SMD:R_0815_2038Metric_Pad1.53x4.00mm_HandSolder" V 9680 4900 50  0001 C CNN
+F 2 "Resistor_SMD:R_0805_2012Metric_Pad1.15x1.40mm_HandSolder" V 9680 4900 50  0001 C CNN
 F 3 "~" H 9750 4900 50  0001 C CNN
 	1    9750 4900
@@
 F 0 "R14" V 9650 1700 50  0000 L CNN
 F 1 "R" V 9650 1600 50  0000 L CNN
-F 2 "Resistor_SMD:R_0815_2038Metric_Pad1.53x4.00mm_HandSolder" V 9480 1700 50  0001 C CNN
+F 2 "Resistor_SMD:R_0805_2012Metric_Pad1.15x1.40mm_HandSolder" V 9480 1700 50  0001 C CNN
 F 3 "~" H 9550 1700 50  0001 C CNN
 	1    9550 1700
@@
 F 0 "R7" H 6570 1696 50  0000 L CNN
 F 1 "R" H 6570 1605 50  0000 L CNN
-F 2 "Resistor_SMD:R_0815_2038Metric_Pad1.53x4.00mm_HandSolder" V 6430 1650 50  0001 C CNN
+F 2 "Resistor_SMD:R_0805_2012Metric_Pad1.15x1.40mm_HandSolder" V 6430 1650 50  0001 C CNN
 F 3 "~" H 6500 1650 50  0001 C CNN
 	1    6500 1650
@@
 F 0 "R8" H 6820 1696 50  0000 L CNN
 F 1 "R" H 6820 1605 50  0000 L CNN
-F 2 "Resistor_SMD:R_0815_2038Metric_Pad1.53x4.00mm_HandSolder" V 6680 1650 50  0001 C CNN
+F 2 "Resistor_SMD:R_0805_2012Metric_Pad1.15x1.40mm_HandSolder" V 6680 1650 50  0001 C CNN
 F 3 "~" H 6750 1650 50  0001 C CNN
 	1    6750 1650
@@
 F 0 "R9" H 7070 1696 50  0000 L CNN
 F 1 "R" H 7070 1605 50  0000 L CNN
-F 2 "Resistor_SMD:R_0815_2038Metric_Pad1.53x4.00mm_HandSolder" V 6930 1650 50  0001 C CNN
+F 2 "Resistor_SMD:R_0805_2012Metric_Pad1.15x1.40mm_HandSolder" V 6930 1650 50  0001 C CNN
 F 3 "~" H 7000 1650 50  0001 C CNN
 	1    7000 1650
@@
 F 0 "R10" H 7320 1696 50  0000 L CNN
 F 1 "R" H 7320 1605 50  0000 L CNN
-F 2 "Resistor_SMD:R_0815_2038Metric_Pad1.53x4.00mm_HandSolder" V 7180 1650 50  0001 C CNN
+F 2 "Resistor_SMD:R_0805_2012Metric_Pad1.15x1.40mm_HandSolder" V 7180 1650 50  0001 C CNN
 F 3 "~" H 7250 1650 50  0001 C CNN
 	1    7250 1650
@@
 F 0 "R6" V 5743 7250 50  0000 C CNN
 F 1 "R" V 5834 7250 50  0000 C CNN
-F 2 "Resistor_SMD:R_0815_2038Metric_Pad1.53x4.00mm_HandSolder" V 5880 7250 50  0001 C CNN
+F 2 "Resistor_SMD:R_0805_2012Metric_Pad1.15x1.40mm_HandSolder" V 5880 7250 50  0001 C CNN
 F 3 "~" H 5950 7250 50  0001 C CNN
 	1    5950 7250
-	0    1    1    0
-$EndComp
-$Comp
-L Connector:Conn_01x01_Male J12
-U 1 1 5F734DCD
-P 5700 6600
-F 0 "J12" V 5762 6644 50  0000 L CNN
-F 1 "Conn_01x01_Male" V 5853 6644 50  0000 L CNN
-F 2 "Connector_PinHeader_2.54mm:PinHeader_1x01_P2.54mm_Vertical" H 5700 6600 50  0001 C CNN
-F 3 "~" H 5700 6600 50  0001 C CNN
-	1    5700 6600
 	0    1    1    0
 $EndComp
@@
 	1    0    0    -1
 $EndComp
-$Comp
-L Connector:Conn_01x01_Male J1
-U 1 1 5F7666DC
-P 900 3400
-F 0 "J1" H 950 3200 50  0000 L CNN
-F 1 "Conn_01x01_Male" H 900 3300 50  0000 L CNN
-F 2 "Connector_PinHeader_2.54mm:PinHeader_1x01_P2.54mm_Vertical" H 900 3400 50  0001 C CNN
-F 3 "~" H 900 3400 50  0001 C CNN
-	1    900  3400
-	1    0    0    -1
-$EndComp
 Wire Wire Line
 	1900 3600 1900 3750
@@
 U 1 1 5F7CB27B
 P 1350 3400
-F 0 "R1" V 1143 3400 50  0000 C CNN
-F 1 "R" V 1234 3400 50  0000 C CNN
-F 2 "Resistor_SMD:R_0815_2038Metric_Pad1.53x4.00mm_HandSolder" V 1280 3400 50  0001 C CNN
+F 0 "R1" V 1300 3550 50  0000 C CNN
+F 1 "R" V 1400 3550 50  0000 C CNN
+F 2 "Resistor_SMD:R_0805_2012Metric_Pad1.15x1.40mm_HandSolder" V 1280 3400 50  0001 C CNN
 F 3 "~" H 1350 3400 50  0001 C CNN
 	1    1350 3400
 	0    1    1    0
 $EndComp
-Wire Wire Line
-	1100 3400 1200 3400
 Wire Wire Line
 	1500 3400 1600 3400
@@
 F 0 "R3" V 4593 4650 50  0000 C CNN
 F 1 "R" V 4684 4650 50  0000 C CNN
-F 2 "Resistor_SMD:R_0815_2038Metric_Pad1.53x4.00mm_HandSolder" V 4730 4650 50  0001 C CNN
+F 2 "Resistor_SMD:R_0805_2012Metric_Pad1.15x1.40mm_HandSolder" V 4730 4650 50  0001 C CNN
 F 3 "~" H 4800 4650 50  0001 C CNN
 	1    4800 4650
@@
 F 0 "R4" V 4593 5100 50  0000 C CNN
 F 1 "R" V 4684 5100 50  0000 C CNN
-F 2 "Resistor_SMD:R_0815_2038Metric_Pad1.53x4.00mm_HandSolder" V 4730 5100 50  0001 C CNN
+F 2 "Resistor_SMD:R_0805_2012Metric_Pad1.15x1.40mm_HandSolder" V 4730 5100 50  0001 C CNN
 F 3 "~" H 4800 5100 50  0001 C CNN
 	1    4800 5100
@@
 F 0 "R12" H 7450 4800 50  0000 C CNN
 F 1 "R" H 7500 4700 50  0000 C CNN
-F 2 "Resistor_SMD:R_0815_2038Metric_Pad1.53x4.00mm_HandSolder" V 7530 4750 50  0001 C CNN
+F 2 "Resistor_SMD:R_0805_2012Metric_Pad1.15x1.40mm_HandSolder" V 7530 4750 50  0001 C CNN
 F 3 "~" H 7600 4750 50  0001 C CNN
 	1    7600 4750
@@
 	6800 5400 6800 5950
 Wire Wire Line
-	6000 5950 6800 5950
+	6000 5950 6350 5950
 Connection ~ 6800 5950
 Wire Wire Line
@@
 Wire Wire Line
 	7300 4800 7350 4800
-$Comp
-L Connector:Conn_01x01_Male J14
-U 1 1 5F6B4498
-P 7350 4150
-F 0 "J14" V 7412 4194 50  0000 L CNN
-F 1 "Conn_01x01_Male" V 7300 3950 50  0000 L CNN
-F 2 "Connector_PinHeader_2.54mm:PinHeader_1x01_P2.54mm_Vertical" H 7350 4150 50  0001 C CNN
-F 3 "~" H 7350 4150 50  0001 C CNN
-	1    7350 4150
-	0    1    1    0
-$EndComp
 Wire Wire Line
 	7600 5350 7600 5450
@@
 P 7600 4400
 F 0 "R11" V 7500 4450 50  0000 C CNN
-F 1 "R" V 7500 4350 50  0000 C CNN
-F 2 "Resistor_SMD:R_0815_2038Metric_Pad1.53x4.00mm_HandSolder" V 7530 4400 50  0001 C CNN
+F 1 "R" V 7500 4300 50  0000 C CNN
+F 2 "Resistor_SMD:R_0805_2012Metric_Pad1.15x1.40mm_HandSolder" V 7530 4400 50  0001 C CNN
 F 3 "~" H 7600 4400 50  0001 C CNN
 	1    7600 4400
@@
 F 0 "J2" H 1050 4650 50  0000 C CNN
 F 1 "Conn_01x04_Male" H 1250 4750 50  0000 C CNN
-F 2 "Connector_PinHeader_2.54mm:PinHeader_1x04_P2.54mm_Vertical" H 1000 5050 50  0001 C CNN
+F 2 "Connector_JST:JST_XH_B4B-XH-A_1x04_P2.50mm_Vertical" H 1000 5050 50  0001 C CNN
 F 3 "~" H 1000 5050 50  0001 C CNN
 	1    1000 5050
@@
 Wire Wire Line
 	6300 5000 6250 5000
-NoConn ~ 6250 5000
+$Comp
+L Device:C C2
+U 1 1 5F6FFCEC
+P 6350 5700
+F 0 "C2" H 6465 5746 50  0000 L CNN
+F 1 "C" H 6465 5655 50  0000 L CNN
+F 2 "Capacitor_SMD:C_0805_2012Metric_Pad1.15x1.40mm_HandSolder" H 6388 5550 50  0001 C CNN
+F 3 "~" H 6350 5700 50  0001 C CNN
+	1    6350 5700
+	1    0    0    -1
+$EndComp
+Wire Wire Line
+	6250 5000 6250 5550
+Wire Wire Line
+	6250 5550 6350 5550
+Wire Wire Line
+	6350 5850 6350 5950
+Connection ~ 6350 5950
+Wire Wire Line
+	6350 5950 6800 5950
+$Comp
+L Connector:Conn_01x03_Male J1
+U 1 1 5F731792
+P 900 3400
+F 0 "J1" H 950 3600 50  0000 C CNN
+F 1 "Conn_01x03_Male" H 1200 3200 50  0000 C CNN
+F 2 "Connector_PinHeader_2.54mm:PinHeader_1x03_P2.54mm_Vertical" H 900 3400 50  0001 C CNN
+F 3 "~" H 900 3400 50  0001 C CNN
+	1    900  3400
+	1    0    0    -1
+$EndComp
+Text Label 5700 6800 0    50   ~ 0
+light_sensor_pin
+Text Label 1100 3300 0    50   ~ 0
+light_sensor_pin
+Text Label 7350 4350 1    50   ~ 0
+timer_pin
+Text Label 1100 3500 0    50   ~ 0
+timer_pin
+Wire Wire Line
+	1100 3400 1200 3400
 $EndSCHEMATC
